File: classdamp.brd (EAGLE design)
At the start: 88.6 x 38.1 mm, 40 parts, among them IC1 78L05, Q1 BS170, Q10 IRF 9Z34N, Q2 BS170, Q7 IRF 530N, Q8 IRF 530N, Q9 IRF 9Z34N

Commit message: removed top layer for production
Routing:
- net GND: track 12.7 -> 0.00 mm
Changed lines of the file:
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@@
 <via x="57.15" y="19.05" extent="1-16" drill="1" diameter="1.6764" shape="square"/>
 <via x="57.15" y="6.35" extent="1-16" drill="1" diameter="1.6764" shape="square"/>
-<wire x1="57.15" y1="19.05" x2="57.15" y2="6.35" width="0.6096" layer="1"/>
 <polygon width="0.254" layer="16" isolate="0.3048">
 <vertex x="88.9" y="22.86"/>

Commit message: adjusted width
Parts:
- moved H1 1.27 mm to (4.45, 32.8)
- moved H2 1.27 mm to (84.5, 32.8)
Routing:
- net +12V: track 39.9 -> 38.8 mm
Other:
- board size 88.6 x 38.1 mm -> 88.6 x 36.8 mm
Changed lines of the file:
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@@
 <plain>
 <wire x1="0" y1="0" x2="88.57" y2="0" width="0" layer="20"/>
-<wire x1="88.57" y1="0" x2="88.57" y2="38.09" width="0" layer="20"/>
-<wire x1="88.57" y1="38.09" x2="0" y2="38.09" width="0" layer="20"/>
-<wire x1="0" y1="38.09" x2="0" y2="0" width="0" layer="20"/>
+<wire x1="88.57" y1="0" x2="88.57" y2="36.82" width="0" layer="20"/>
+<wire x1="88.57" y1="36.82" x2="0" y2="36.82" width="0" layer="20"/>
+<wire x1="0" y1="36.82" x2="0" y2="0" width="0" layer="20"/>
 <text x="7.62" y="19.05" size="1.778" layer="16" font="vector" ratio="14" rot="MR270">D-Amp</text>
 <text x="4.445" y="30.48" size="1.778" layer="16" font="vector" ratio="15" rot="MR270">Signal Generator</text>
 <dimension x1="0" y1="39.37" x2="88.9" y2="39.37" x3="44.45" y3="44.45" textsize="1.778" textratio="15" layer="47"/>
-<dimension x1="89.84" y1="0" x2="89.84" y2="38.09" x3="96.52" y3="19.045" textsize="1.778" textratio="15" layer="47" precision="1"/>
+<dimension x1="89.84" y1="0" x2="89.84" y2="36.82" x3="96.52" y3="18.41" textsize="1.778" textratio="15" layer="47" precision="1"/>
 <dimension x1="84.455" y1="33.655" x2="4.445" y2="33.655" x3="44.45" y3="40.64" textsize="1.778" textratio="15" layer="47" precision="1"/>
-<dimension x1="84.455" y1="4.045" x2="84.455" y2="34.055" x3="92.71" y3="19.05" textsize="1.778" textratio="15" layer="47" precision="1"/>
+<dimension x1="84.455" y1="4.045" x2="84.455" y2="32.785" x3="92.71" y3="18.415" textsize="1.778" layer="20"/>
 </plain>
 <attributes>
@@
 <attribute name="OC_FARNELL" value="unknown" x="81.28" y="12.7" size="1.778" layer="27" rot="R270" display="off"/>
 </element>
-<element name="H2" library="holes" package="3,2" value="MOUNT-HOLE3.2" x="84.455" y="34.055" rot="MR0"/>
+<element name="H2" library="holes" package="3,2" value="MOUNT-HOLE3.2" x="84.455" y="32.785" rot="MR0"/>
 <element name="H3" library="holes" package="3,2" value="MOUNT-HOLE3.2" x="84.455" y="4.045"/>
 <element name="H4" library="holes" package="3,2" value="MOUNT-HOLE3.2" x="4.445" y="4.045"/>
-<element name="H1" library="holes" package="3,2" value="MOUNT-HOLE3.2" x="4.445" y="34.055"/>
+<element name="H1" library="holes" package="3,2" value="MOUNT-HOLE3.2" x="4.445" y="32.785"/>
 <element name="JP2" library="pinhead" package="1X03" value="ISP1" x="38.1" y="10.16" rot="R90"/>
 <element name="JP8" library="pinhead" package="1X03" value="ISP2" x="38.1" y="27.94" rot="R270"/>
@@
 <vertex x="73.9775" y="25.7175"/>
 </polygon>
-<wire x1="76.2" y1="35.56" x2="83.82" y2="27.94" width="1.016" layer="16"/>
+<wire x1="77.47" y1="34.29" x2="83.82" y2="27.94" width="1.016" layer="16"/>
 <wire x1="83.82" y1="27.94" x2="83.82" y2="20.955" width="1.016" layer="16"/>
-<wire x1="54.61" y1="34.29" x2="55.88" y2="34.29" width="1.016" layer="16"/>
-<wire x1="55.88" y1="34.29" x2="57.15" y2="35.56" width="1.016" layer="16"/>
-<wire x1="57.15" y1="35.56" x2="76.2" y2="35.56" width="1.016" layer="16"/>
+<wire x1="54.61" y1="34.29" x2="77.47" y2="34.29" width="1.016" layer="16"/>
 <contactref element="X2" pad="2"/>
 <contactref element="C2" pad="1"/>
